File: ac-power-monitor.kicad_pcb (KiCad board)
At the start: 2 copper layers, 100 x 50 mm, 65 parts, among them J1 CONN2, J2 CONN2, J3 CONN2, J4 CONN8, J5 CONN6, P1 FASTON_1, P2 FASTON_1, P3 FASTON_1, P4 FASTON_1, U1 AZ1117CH-3.3TRG1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

Commit message: Release revision A schematic, board, and BOM. Update picture to show revision A board. Remove X1 rework instructions from README.md.
Parts:
- removed the MTG-HOLE-M2-RING-5MM at (198.5, 78.0)
- removed the MTG-HOLE-M2-RING-5MM at (198.5, 95.1)
- removed R14, R15: 10K, mods:RC0603
- removed R16: 0, mods:RC0805
- added MTG-HOLE-M2-RING-5MM: VAL**, mods:MTG-HOLE-M2-RING-5MM, F.Cu at (198.4, 78.0)
- added MTG-HOLE-M2-RING-5MM: VAL**, mods:MTG-HOLE-M2-RING-5MM, F.Cu at (198.4, 95.1)
- moved R17 31.1 mm to (171.3, 117.7)
- moved Sym 0.79 mm to (144.8, 90.8)
Connections:
- net Net-(J4-Pad7) renamed /WIFI/GPIO16
- J4 pad 2: ~CS -> (no net)
- J4 pad 3: IRQ -> (no net)
- J5 pad 3: (no net) -> /WIFI/SPWR
- R17 pad 1: Net-(R15-Pad2) -> +3.3V
- R17 pad 2: GND -> /WIFI/SPWR
- U2 pad 1: Net-(R14-Pad2) -> GND
- U2 pad 20: IRQ -> (no net)
- U2 pad 24: ~CS -> GND
- U2 pad 28: Net-(R15-Pad2) -> +3.3V
- U3 pad 13: IRQ -> (no net)
- U3 pad 14: ~CS -> (no net)
Routing:
- net ~CS: track 86.2 -> 0.00 mm, vias 7 -> 0
- net IRQ: track 68.9 -> 0.00 mm, vias 6 -> 0
- net +3.3V: track 147.5 -> 168.8 mm, vias 6 -> 8
- net Net-(R14-Pad2): track 9.52 -> 0.00 mm
- net Net-(R15-Pad2): track 5.61 -> 0.00 mm
- net /WIFI/SPWR: track 0.00 -> 5.29 mm
- net GND: track 120.9 -> 121.7 mm
Other:
- board text added: "RESET"
- board text added: "WIFI AC POWER MONITOR 66-100105 A COPYRIGHT 2015 STEPHEN RODGERS HWSTAR"
- board text removed: "WIFI AC POWER MONITOR 66-100105 X1 COPYRIGHT 2015 STEPHEN RODGERS HWSTAR"
