File: metrology.sch (KiCad schematic (older format))
At the start: 16 parts, among them U2 90E24PYGI, Y1 8.192MHz

Commit message: Release revision A schematic, board, and BOM. Update picture to show revision A board. Remove X1 rework instructions from README.md.
Parts:
- removed R14, R15: 10K, mods:RC0603, symbol R_US
- removed R16, R17: 0, mods:RC0805, symbol R_US
Connections:
- net ~CS is gone; now on net GND: U2.24 (~CS)
- net +3.3V: now also U2.28 (MMD0)
- net GND: now also U2.1 (MMD1)
- net IRQ: no longer names the net of U2.20 (IRQ)
- no-connect marks 0 -> 1
Other:
- note added: "MODE : L LINE MODE\n"
Changed lines of the file:
@@
-$EndComp
-$Comp
-L R_US R14
-U 1 1 55C7E1E9
-P 7050 2300
-F 0 "R14" V 7130 2300 50  0000 C CNN
-F 1 "10K" V 6970 2300 50  0000 C CNN
-F 2 "mods:RC0603" H 7050 2300 60  0001 C CNN
-F 3 "" H 7050 2300 60  0000 C CNN
-F 4 "800010-103" V 7050 2300 60  0001 C CNN "PartNumber"
-	1    7050 2300
-	1    0    0    -1
 $EndComp
 $Comp
@@
 	1    0    0    -1
 $EndComp
-$Comp
-L GND_US #PWR011
-U 1 1 55C7E389
-P 7450 3200
-F 0 "#PWR011" H 7430 3070 30  0001 C CNN
-F 1 "GND_US" H 7440 3110 30  0001 C CNN
-F 2 "" H 7450 3200 60  0000 C CNN
-F 3 "" H 7450 3200 60  0000 C CNN
-	1    7450 3200
-	1    0    0    -1
-$EndComp
 Text GLabel 6300 3550 2    60   Input ~ 0
 SCLK
@@
 Text GLabel 6300 3750 2    60   Input ~ 0
 SDI
-Text GLabel 6650 3850 2    60   Input ~ 0
-~CS
-Text GLabel 6300 3950 2    60   Input ~ 0
-IRQ
 $Comp
 L TESTPINTPSQ025 TP2
@@
 $EndComp
 $Comp
-L GND_US #PWR012
+L GND_US #PWR011
 U 1 1 55C7EC21
 P 5150 2650
-F 0 "#PWR012" H 5130 2520 30  0001 C CNN
+F 0 "#PWR011" H 5130 2520 30  0001 C CNN
 F 1 "GND_US" H 5140 2560 30  0001 C CNN
 F 2 "" H 5150 2650 60  0000 C CNN
@@
 $EndComp
 $Comp
-L GND_US #PWR013
+L GND_US #PWR012
 U 1 1 55C7EDE2
 P 4550 5450
-F 0 "#PWR013" H 4530 5320 30  0001 C CNN
+F 0 "#PWR012" H 4530 5320 30  0001 C CNN
 F 1 "GND_US" H 4540 5360 30  0001 C CNN
 F 2 "" H 4550 5450 60  0000 C CNN
@@
 $EndComp
 $Comp
-L GND_US #PWR014
+L GND_US #PWR013
 U 1 1 55C7F0A9
 P 4150 5450
-F 0 "#PWR014" H 4130 5320 30  0001 C CNN
+F 0 "#PWR013" H 4130 5320 30  0001 C CNN
 F 1 "GND_US" H 4140 5360 30  0001 C CNN
 F 2 "" H 4150 5450 60  0000 C CNN
@@
 $EndComp
 $Comp
-L GND_US #PWR015
+L GND_US #PWR014
 U 1 1 55C80A38
 P 3650 5450
-F 0 "#PWR015" H 3630 5320 30  0001 C CNN
+F 0 "#PWR014" H 3630 5320 30  0001 C CNN
 F 1 "GND_US" H 3640 5360 30  0001 C CNN
 F 2 "" H 3650 5450 60  0000 C CNN
@@
 $EndComp
 $Comp
-L GND_US #PWR016
+L GND_US #PWR015
 U 1 1 55C8E301
 P 4500 4450
-F 0 "#PWR016" H 4480 4320 30  0001 C CNN
+F 0 "#PWR015" H 4480 4320 30  0001 C CNN
 F 1 "GND_US" H 4490 4360 30  0001 C CNN
 F 2 "" H 4500 4450 60  0000 C CNN
@@
 ISAMPLEN
 $Comp
-L R_US R16
-U 1 1 55C92157
-P 7050 2900
-F 0 "R16" V 7130 2900 50  0000 C CNN
-F 1 "0" V 6970 2900 50  0000 C CNN
-F 2 "mods:RC0805" H 7050 2900 60  0001 C CNN
-F 3 "" H 7050 2900 60  0000 C CNN
-F 4 "800011-000" V 7050 2900 60  0001 C CNN "PartNumber"
-	1    7050 2900
-	1    0    0    -1
-$EndComp
-$Comp
-L R_US R17
-U 1 1 55C921A7
-P 7450 2900
-F 0 "R17" V 7530 2900 50  0000 C CNN
-F 1 "0" V 7370 2900 50  0000 C CNN
-F 2 "mods:RC0805" H 7450 2900 60  0001 C CNN
-F 3 "" H 7450 2900 60  0000 C CNN
-F 4 "800011-000" V 7450 2900 60  0001 C CNN "PartNumber"
-	1    7450 2900
-	1    0    0    -1
-$EndComp
-$Comp
-L R_US R15
-U 1 1 55C922A9
-P 7450 2300
-F 0 "R15" V 7530 2300 50  0000 C CNN
-F 1 "10K" V 7370 2300 50  0000 C CNN
-F 2 "mods:RC0603" H 7450 2300 60  0001 C CNN
-F 3 "" H 7450 2300 60  0000 C CNN
-F 4 "800010-103" V 7450 2300 60  0001 C CNN "PartNumber"
-	1    7450 2300
-	1    0    0    -1
-$EndComp
-$Comp
-L PWR_FLAG #FLG017
+L PWR_FLAG #FLG016
 U 1 1 55C9312D
 P 5850 1700
-F 0 "#FLG017" H 5850 1795 50  0001 C CNN
+F 0 "#FLG016" H 5850 1795 50  0001 C CNN
 F 1 "PWR_FLAG" H 5850 1880 50  0000 C CNN
 F 2 "" H 5850 1700 60  0000 C CNN
@@
 $EndComp
 $Comp
-L +3.3V #PWR018
+L +3.3V #PWR017
 U 1 1 55CA6A61
 P 3850 1250
-F 0 "#PWR018" H 3850 1210 30  0001 C CNN
+F 0 "#PWR017" H 3850 1210 30  0001 C CNN
 F 1 "+3.3V" H 3850 1360 30  0000 C CNN
 F 2 "" H 3850 1250 60  0000 C CNN
@@
 $EndComp
 Wire Wire Line
-	7450 2050 7450 2100
+	7450 2050 7450 2650
 Wire Wire Line
 	5750 2050 7450 2050
@@
 Connection ~ 6300 2050
 Wire Wire Line
-	7050 2100 7050 2050
-Connection ~ 7050 2050
-Wire Wire Line
 	6300 3050 5850 3050
 Wire Wire Line
@@
 	6050 2950 6050 2050
 Wire Wire Line
-	7050 2500 7050 2700
-Wire Wire Line
-	7450 2500 7450 2700
-Wire Wire Line
 	5850 3250 6450 3250
 Wire Wire Line
@@
 Wire Wire Line
 	6450 2550 7050 2550
-Connection ~ 7050 2550
 Wire Wire Line
 	5850 3350 6550 3350
@@
 Wire Wire Line
 	6550 2650 7450 2650
-Connection ~ 7450 2650
-Wire Wire Line
-	7050 3100 7050 3200
-Wire Wire Line
-	7450 3100 7450 3200
+Wire Wire Line
+	7050 2550 7050 3200
 Wire Wire Line
 	5850 3650 6650 3650
 Wire Wire Line
 	5850 3750 6300 3750
-Wire Wire Line
-	5850 3850 6650 3850
 Wire Wire Line
 	5850 3550 6300 3550
@@
 	3100 3300 2650 3300
 Connection ~ 5850 2500
-Wire Wire Line
-	5850 3950 6300 3950
 Wire Wire Line
 	5350 2050 5150 2050
@@
 Wire Wire Line
 	3850 1500 3850 1250
+$Comp
+L GND_US #PWR018
+U 1 1 5601E892
+P 6650 4000
+F 0 "#PWR018" H 6630 3870 30  0001 C CNN
+F 1 "GND_US" H 6640 3910 30  0001 C CNN
+F 2 "" H 6650 4000 60  0000 C CNN
+F 3 "" H 6650 4000 60  0000 C CNN
+	1    6650 4000
+	1    0    0    -1
+$EndComp
+Wire Wire Line
+	5850 3850 6650 3850
+Wire Wire Line
+	6650 3850 6650 4000
+Text Notes 7150 2900 0    60   ~ 0
+MODE : L LINE MODE\n
+NoConn ~ 5850 3950
 $EndSCHEMATC
